File: EAGLE Files/Buggy Motor Board.brd (EAGLE design)
At the start: 100 x 80 mm, 19 parts, among them IC1 ILD213T, IC2 ILD213T

Commit message: Added shift register (TEST)
Parts:
- added IC3: 74HC595D, 74xx-eu:SO16
Connections:
- new net VCC: IC3.16
- net GND: now also IC3.8
Changed lines of the file:
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@@
 <element name="U$4" library="SparkFun-AnalogIC" package="SOT23-6-MCP4725" value="DAC_MCP4725SOT-CP" x="8.89" y="45.72" rot="R90"/>
 <element name="U$5" library="SparkFun-Connectors" package="RJ45-8" value="RJ45-8PTH" x="21.59" y="3.81"/>
+<element name="IC3" library="74xx-eu" package="SO16" value="74HC595D" x="7.62" y="-12.7"/>
 </elements>
 <signals>
@@
 <contactref element="U$3" pad="2"/>
 <contactref element="U$5" pad="1"/>
+<contactref element="IC3" pad="8"/>
 <wire x1="21.59" y1="52.07" x2="36.83" y2="57.15" width="0" layer="19" extent="1-1"/>
 <wire x1="10.1901" y1="45.72" x2="21.59" y2="52.07" width="0" layer="19" extent="1-1"/>
@@
 <wire x1="6.12" y1="54.61" x2="10.1901" y2="45.72" width="0" layer="19" extent="1-1"/>
 <wire x1="17.145" y1="10.16" x2="5.0038" y2="23.495" width="0" layer="19" extent="1-1"/>
+<wire x1="12.065" y1="-15.7734" x2="17.145" y2="10.16" width="0" layer="19" extent="1-1"/>
 </signal>
 <signal name="AGND">
@@
 <wire x1="5.0038" y1="24.765" x2="21.59" y2="31.75" width="0" layer="19" extent="1-1"/>
 </signal>
+<signal name="VCC">
+<contactref element="IC3" pad="16"/>
+</signal>
 </signals>
