File: EAGLE Files/Red Buggy 2015.brd (EAGLE design)
At the start: 100 x 80 mm, 13 parts, among them K1 CB1A-P-12V, K2 CB1A-P-12V

Commit message: Tweak for Red Buggy
Removed IMU, second opto-coupler, shift registers;  added connectors for
Curtis motor controllers
Connections:
- net MS2: now also JP2.3
Changed lines of the file:
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@@
 <contactref element="MODE-R" pad="2"/>
 <contactref element="JP1" pad="3"/>
-<wire x1="-54.8894" y1="39.3954" x2="25.4" y2="45.72" width="0" layer="19" extent="1-1"/>
+<contactref element="JP2" pad="3"/>
+<wire x1="-54.8894" y1="39.3954" x2="-72.39" y2="-6.35" width="0" layer="19" extent="1-1"/>
+<wire x1="25.4" y1="45.72" x2="-54.8894" y2="39.3954" width="0" layer="19" extent="1-1"/>
 </signal>
 <signal name="ILOCK">
