File: EAGLE Files/Red Buggy 2015.sch (EAGLE design)
At the start: 13 parts, among them K1 CB1A-P-12V, K2 CB1A-P-12V

Commit message: Tweak for Red Buggy
Removed IMU, second opto-coupler, shift registers;  added connectors for
Curtis motor controllers
Connections:
- net MS2: now also JP2.3
Changed lines of the file:
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@@
 <wire x1="160.02" y1="60.96" x2="162.56" y2="63.5" width="0.1524" layer="91"/>
 <label x="154.94" y="60.96" size="1.778" layer="95"/>
+<pinref part="JP2" gate="A" pin="3"/>
+<wire x1="160.02" y1="60.96" x2="149.86" y2="60.96" width="0.1524" layer="91"/>
 </segment>
 </net>
